File: TekV2/circuit/TekV2.brd (EAGLE design)
At the start: 100 x 80 mm, 7 parts, among them IC1 74HC74N, IC2 74LS32N

Commit message: fixed connection of diode
Connections:
- net N$2: now also IC1.8; no longer IC1.9
Changed lines of the file:
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@@
 <signal name="N$2">
 <contactref element="D1" pad="C"/>
-<contactref element="IC1" pad="9"/>
-<wire x1="53.34" y1="24.13" x2="35.56" y2="12.7" width="0" layer="19" extent="1-1"/>
+<contactref element="IC1" pad="8"/>
+<wire x1="35.56" y1="10.16" x2="53.34" y2="24.13" width="0" layer="19" extent="1-1"/>
 </signal>
 <signal name="PS2DAT">
